Commit message: adjustments for real robot
Conflicts:
	catkin_ws/src/PioneerModel/p3dx_description/launch/everything.launch

File: catkin_ws/src/PioneerModel/p3dx_description/urdf/pioneer3dx.xacro (robot description, xacro)
@@ -200,5 +200,5 @@
   <joint name="camera_joint" type="fixed">
     <axis xyz="0 0 0" />
-    <origin xyz="${camera_link} 0.0 -0.135" rpy="0 0 0"/>
+    <origin xyz="${camera_link} 0.0 0.05" rpy="0 0 0"/>
     <parent link="front_sonar"/>
     <child link="camera_link"/>

Commit message: stuff which works in real life
Conflicts:
	catkin_ws/src/PioneerModel/p3dx_description/launch/everything.launch

File: catkin_ws/src/PioneerModel/p3dx_description/urdf/pioneer3dx.xacro (robot description, xacro)
@@ -239,4 +239,11 @@
   <link name="camera_depth_frame">
   </link>
+  <joint name="kinect2_ir_optical_joint" type="fixed">
+    <origin rpy="-1.571 0 -1.571"/>
+    <parent link="camera_link"/>
+    <child link="kinect2_ir_optical_frame"/>
+  </joint>
+  <link name="kinect2_ir_optical_frame">
+  </link>
 	<xacro:property name="camera_link" value="0.05" /> <!-- Size of square 'camera' box -->
 </robot>
